Commit message: added nav

File: Ros/roboin_description/urdf/roboin.xacro (robot description, xacro)
@@ -6,5 +6,5 @@
     <parent link="base_footprint"/>
     <child link="base_link" />
-    <origin xyz="0 0 0.1" rpy="0 0 0"/>
+    <origin xyz="0.1 0 0.1" rpy="0 0 0"/>
   </joint>
 <!--base_link-->
@@ -111,4 +111,12 @@
     </collision>
   </link>
+<!--IMU-->
+  <joint name="imu_joint" type="fixed">
+    <parent link="base_link"/>
+    <child link="imu_link"/>
+    <origin xyz="0 0 0.05" rpy="0 0 0"/>
+  </joint>
+  <link name="imu_link">
+  </link>
 <!--lidar-->
   <joint name="scan_joint" type="fixed">

File: Ros/roboin_description/urdf/roboin_gazebo_plugins.xacro (robot description, xacro)
@@ -47,5 +47,5 @@
       <wheelSeparation>0.23</wheelSeparation>
       <wheelDiameter>0.06</wheelDiameter>
-      <wheelAcceleration>1</wheelAcceleration>
+      <wheelAcceleration>0</wheelAcceleration>
       <wheelTorque>5</wheelTorque>
       <rosDebugLevel>na</rosDebugLevel>
@@ -57,5 +57,5 @@
       <pose>0 0 0 0 0 0</pose>
       <visualize>$(arg laser_visual)</visualize>
-      <update_rate>5</update_rate>
+      <update_rate>10</update_rate>
       <ray>
         <scan>
