Commit message: roborts path planning in gazebo

File: Ros/roborts/roborts_gazebo/urdf/robomaster.xacro (robot description, xacro)
@@ -42,8 +42,8 @@
   <joint name="scan_joint" type="fixed">
     <parent link="base_link"/>
-    <child link="base_scan"/>
+    <child link="base_laser_link"/>
     <origin xyz="-0.2 0 0.075" rpy="0 0 0"/>
   </joint>
-  <link name="base_scan">
+  <link name="base_laser_link">
     <visual>
       <origin xyz="0 0 0" rpy="0 0 0"/>

File: Ros/roborts/roborts_gazebo/urdf/robomaster_gazebo.xacro (robot description, xacro)
@@ -4,5 +4,5 @@
   <xacro:arg name="camera_visual" default="false"/>
   <xacro:arg name="imu_visual"    default="false"/>
-  <gazebo reference="base_scan">
+  <gazebo reference="base_laser_link">
     <material>Gazebo/FlatBlack</material>
     <sensor type="ray" name="lidar">
@@ -32,5 +32,5 @@
       <plugin name="gazebo_ros_lds_lfcd_controller" filename="libgazebo_ros_laser.so">
         <topicName>scan</topicName>
-        <frameName>base_scan</frameName>
+        <frameName>base_laser_link</frameName>
       </plugin>
     </sensor>
