Commit message: roborts update

File: Ros_old/roborts/roborts_gazebo/urdf/robomaster_ai.gazebo.xacro (robot description, xacro)
@@ -27,4 +27,8 @@
   </gazebo>
   <gazebo reference="led_Link">
+    <material>Gazebo/Red</material>
+    <turnGravityOff>false</turnGravityOff>
+  </gazebo>
+  <gazebo reference="yaw_Link">
     <material>Gazebo/Red</material>
     <turnGravityOff>false</turnGravityOff>
@@ -124,3 +128,9 @@
     </plugin>
   </gazebo>
+   <gazebo>
+    <plugin name="roborts_shooter" filename="libroborts_shooter_plugin.so">
+      <gimbal_link>pitch_Link</gimbal_link>
+      <reference_frame>map</reference_frame>
+    </plugin>
+  </gazebo>
 </robot>

File: Ros_old/roborts/roborts_gazebo/urdf/robomaster_ai.xacro (robot description, xacro)
@@ -1,5 +1,7 @@
 <?xml version="1.0"?>
 <robot xmlns:xacro="http://www.ros.org/wiki/xacro" name="robomaster_ai">
-  <xacro:include filename="$(find roborts_gazebo)/urdf/robomaster_ai_gazebo.xacro"/>
+  <xacro:include filename="$(find roborts_gazebo)/urdf/robomaster_ai.gazebo.xacro"/>
+  <xacro:include filename="$(find roborts_gazebo)/urdf/robomaster_ai.trans.xacro"/>
+  <xacro:include filename="$(find roborts_gazebo)/urdf/robomaster_ai.bullet.xacro"/>
   <link name="base_footprint"/>
   <joint name="base_joint" type="fixed">
@@ -305,13 +307,4 @@
       </material>
     </visual>
-    <collision>
-      <origin
-        xyz="0 0 0"
-        rpy="0 0 0" />
-      <geometry>
-        <mesh
-          filename="package://roborts_gazebo/meshes/pitch_Link.STL" />
-      </geometry>
-    </collision>
   </link>
   <joint
@@ -492,23 +485,3 @@
       xyz="0 0 0" />
   </joint>
-  <transmission name="base_link_to_yaw_joint_trans">
-    <type>transmission_interface/SimpleTransmission</type>
-    <joint name="base_link_to_yaw_joint">
-      <hardwareInterface>hardware_interface/EffortJointInterface</hardwareInterface>
-    </joint>
-    <actuator name="base_link_to_yaw_joint_motor">
-      <mechanicalReduction>1</mechanicalReduction>
-      <hardwareInterface>EffortJointInterface</hardwareInterface>
-    </actuator>
-  </transmission>
-  <transmission name="base_link_to_pitch_joint_trans">
-    <type>transmission_interface/SimpleTransmission</type>
-    <joint name="base_link_to_pitch_joint">
-      <hardwareInterface>hardware_interface/EffortJointInterface</hardwareInterface>
-    </joint>
-    <actuator name="base_link_to_pitch_joint_motor">
-      <mechanicalReduction>1</mechanicalReduction>
-      <hardwareInterface>EffortJointInterface</hardwareInterface>
-    </actuator>
-  </transmission>
 </robot>

File: Ros_old/roborts/roborts_gazebo/urdf/robomaster_gazebo.xacro (robot description, xacro)
@@ -89,3 +89,9 @@
    </plugin>
  </gazebo>
+ <gazebo>
+  <plugin name="roborts_shooter" filename="libroborts_shooter_plugin.so">
+    <gimbal_link>pitch_Link</gimbal_link>
+    <reference_frame>map</reference_frame>
+  </plugin>
+ </gazebo>
 </robot>

Commit message: update roborts

File: Ros_old/roborts/roborts_gazebo/urdf/robomaster_ai.gazebo.xacro (robot description, xacro)
@@ -2,8 +2,8 @@
 <robot>
   <!-- materials -->
-  <gazebo reference="base_link">
+  <!--<gazebo reference="base_link">
     <material>Gazebo/Black</material>
     <turnGravityOff>false</turnGravityOff>
-  </gazebo>
+  </gazebo>-->
   <gazebo reference="fr_wheel_Link">
     <material>Gazebo/Black</material>
@@ -38,5 +38,5 @@
     <sensor type="ray" name="head_hokuyo_sensor">
       <pose>2000 2000 2000 0 0 0</pose>
-      <visualize>true</visualize>
+      <visualize>false</visualize>
       <update_rate>40</update_rate>
       <ray>
@@ -131,5 +131,7 @@
     <plugin name="roborts_shooter" filename="libroborts_shooter_plugin.so">
       <gimbal_link>pitch_Link</gimbal_link>
+      <fake_link>fake_link</fake_link>
       <reference_frame>map</reference_frame>
+      <force>2000.0</force>
     </plugin>
   </gazebo>

File: Ros_old/roborts/roborts_gazebo/urdf/robomaster_ai.xacro (robot description, xacro)
@@ -3,5 +3,4 @@
   <xacro:include filename="$(find roborts_gazebo)/urdf/robomaster_ai.gazebo.xacro"/>
   <xacro:include filename="$(find roborts_gazebo)/urdf/robomaster_ai.trans.xacro"/>
-  <xacro:include filename="$(find roborts_gazebo)/urdf/robomaster_ai.bullet.xacro"/>
   <link name="base_footprint"/>
   <joint name="base_joint" type="fixed">
@@ -29,5 +28,5 @@
         rpy="0 0 0" />
       <geometry>
-        <mesh filename="package://roborts_gazebo/meshes/base_link.STL" />
+        <mesh filename="package://roborts_gazebo/meshes/base_link_2.STL" />
       </geometry>
       <material name="">
@@ -307,4 +306,25 @@
       </material>
     </visual>
+  </link>
+  <joint name="fake_joint" type="continuous">
+    <parent link="pitch_Link"/>
+    <child link="fake_link"/>
+    <origin xyz="0.2 0 0" rpy="0 0 0"/>
+  </joint>
+  <link name="fake_link">
+    <inertial>
+      <origin xyz="0 0 0" rpy="0 0 0"/>
+      <mass value="0.1"/>
+      <inertia ixx="0.0004"  ixy="0"  ixz="0" iyy="0.0004" iyz="0" izz="0.0004" />
+    </inertial>
+    <!--<visual>
+      <origin xyz="0 0 0" rpy="0 0 0"/>
+      <geometry>
+        <sphere radius="0.02"/>
+      </geometry>
+      <material name="white">
+        <color rgba="1.0 1.0 1.0 1.0"/>
+      </material>
+    </visual>-->
   </link>
   <joint
@@ -356,5 +376,5 @@
       </material>
     </visual>
-    <collision>
+    <!--<collision>
       <origin
         xyz="0 0 0"
@@ -364,5 +384,5 @@
           filename="package://roborts_gazebo/meshes/camera_Link.STL" />
       </geometry>
-    </collision>
+    </collision>-->
   </link>
   <joint
@@ -409,5 +429,5 @@
       </material>
     </visual>
-    <collision>
+    <!--<collision>
       <origin
         xyz="0 0 0"
@@ -417,5 +437,5 @@
           filename="package://roborts_gazebo/meshes/laser_Link.STL" />
       </geometry>
-    </collision>
+    </collision>-->
   </link>
   <joint

File: Ros_old/roborts/roborts_gazebo/urdf/robomaster_gazebo.xacro (robot description, xacro)
@@ -89,9 +89,10 @@
    </plugin>
  </gazebo>
- <gazebo>
+ <!--<gazebo>
   <plugin name="roborts_shooter" filename="libroborts_shooter_plugin.so">
     <gimbal_link>pitch_Link</gimbal_link>
+    <fake_link>fake_link</fake_link>
     <reference_frame>map</reference_frame>
   </plugin>
- </gazebo>
+ </gazebo>-->
 </robot>
