Commit message: gazebo robot model and particle shooter update

File: Ros_old/roborts/roborts_gazebo/urdf/roborts.xacro (robot description, xacro)
@@ -1,27 +1,38 @@
-<robot
-  name="roborts">
+<?xml version="1.0"?>
+<robot xmlns:xacro="http://www.ros.org/wiki/xacro" name="roborts">
+  <xacro:include filename="$(find roborts_gazebo)/urdf/roborts.gazebo.xacro"/>
+  <xacro:include filename="$(find roborts_gazebo)/urdf/roborts.trans.xacro"/>
   <link name="base_footprint"/>
   <joint name="base_joint" type="fixed">
     <parent link="base_footprint"/>
     <child link="base_link" />
-    <origin xyz="0 0 0" rpy="0 0 0"/>
-  </joint>
-  <link
-    name="base_link">
-    <inertial>
-      <origin
-        xyz="0.0911703133114876 0.532603557688202 -0.0712304066002232"
-        rpy="0 0 0" />
-      <mass
-        value="12.50345535509228" />
-      <inertia
-        ixx="0.0696144181432877"
-        ixy="-4.10992920734967E-06"
-        ixz="5.83569660872888E-05"
-        iyy="0.0299049539551884"
-        iyz="-0.00505054745740228"
-        izz="0.084986264822875" />
-    </inertial>
-    <visual>
+    <origin xyz="0.1 0 0.1" rpy="0 0 0"/>
+  </joint>
+  <link name="base_link">
+    <inertial>
+      <origin
+        xyz="-0.025782 -8.2911E-05 0.025311"
+        rpy="0 0 0" />
+      <mass value="7.625" />
+      <inertia
+        ixx="0.10311"
+        ixy="-9.0391E-05"
+        ixz="0.0071078"
+        iyy="0.24575"
+        iyz="2.1083E-05"
+        izz="0.32438" />
+    </inertial>
+    <visual>
+      <origin
+        xyz="-0.536 -0.097 -0.02"
+        rpy="1.5708 0 1.5708" />
+      <geometry>
+        <mesh filename="package://roborts_gazebo/meshes/base_link.STL" />
+      </geometry>
+      <material name="">
+        <color rgba="0.79216 0.81961 0.93333 1" />
+      </material>
+    </visual>
+    <!--<collision>
       <origin
         xyz="0 0 0"
@@ -31,8 +42,30 @@
           filename="package://roborts_gazebo/meshes/base_link.STL" />
       </geometry>
-      <material
-        name="">
-        <color
-          rgba="0.792156862745098 0.819607843137255 0.933333333333333 1" />
+    </collision>-->
+  </link>
+  <link name="fl_wheel_Link">
+    <inertial>
+      <origin
+        xyz="-5.232E-06 0.014616 -9.0427E-06"
+        rpy="0 0 0" />
+      <mass
+        value="0.86078" />
+      <inertia
+        ixx="0.0015361"
+        ixy="1.6456E-06"
+        ixz="-2.0131E-06"
+        iyy="0.002844"
+        iyz="-9.5351E-07"
+        izz="0.0015337" />
+    </inertial>
+    <visual>
+      <origin
+        xyz="0 0 0"
+        rpy="1.5708 0 1.5708" />
+      <geometry>
+        <mesh filename="package://roborts_gazebo/meshes/Front_Left_Wheel.STL" />
+      </geometry>
+      <material name="">
+        <color rgba="0.79216 0.81961 0.93333 1" />
       </material>
     </visual>
@@ -40,39 +73,42 @@
       <origin
         xyz="0 0 0"
-        rpy="0 0 0" />
-      <geometry>
-        <mesh
-          filename="package://roborts_gazebo/meshes/base_link.STL" />
+        rpy="1.5708 0 1.5708"/>
+      <geometry>
+        <mesh filename="package://roborts_gazebo/meshes/Front_Left_Wheel.STL" />
       </geometry>
     </collision>
   </link>
-  <link
-    name="Front_Right_Wheel">
-    <inertial>
-      <origin
-        xyz="-0.023927 -4.9049E-06 -4.7297E-07"
-        rpy="0 0 0" />
-      <mass
-        value="0.21911" />
-      <inertia
-        ixx="0.00087242"
-        ixy="-2.3396E-08"
-        ixz="2.3653E-07"
-        iyy="0.00045739"
-        iyz="-5.7565E-08"
-        izz="0.00045797" />
-    </inertial>
-    <visual>
-      <origin
-        xyz="0 0 0"
-        rpy="0 0 0" />
-      <geometry>
-        <mesh
-          filename="package://roborts_gazebo/meshes/Front_Right_Wheel.STL" />
-      </geometry>
-      <material
-        name="">
-        <color
-          rgba="0.79216 0.81961 0.93333 1" />
+  <joint
+    name="base_link_to_fl_wheel_joint"
+    type="fixed">
+    <origin
+      xyz="0.21194 -0.1709 0.0022"
+      rpy="4.8881E-16 -3.6891E-17 -3.1416" />
+    <parent link="base_link" />
+    <child link="fl_wheel_Link" />
+  </joint>
+  <link name="fr_wheel_Link">
+    <inertial>
+      <origin
+        xyz="0.00010086 -0.014551 4.8285E-05"
+        rpy="0 0 0" />
+      <mass value="0.86078" />
+      <inertia
+        ixx="0.0015355"
+        ixy="4.8831E-07"
+        ixz="1.8067E-06"
+        iyy="0.002844"
+        iyz="9.4618E-08"
+        izz="0.0015338" />
+    </inertial>
+    <visual>
+      <origin
+        xyz="0 0 0"
+        rpy="1.5708 0 1.5708"/>
+      <geometry>
+        <mesh filename="package://roborts_gazebo/meshes/Front_Right_Wheel.STL" />
+      </geometry>
+      <material name="">
+        <color rgba="0.79216 0.81961 0.93333 1" />
       </material>
     </visual>
@@ -80,196 +116,109 @@
       <origin
         xyz="0 0 0"
-        rpy="0 0 0" />
-      <geometry>
-        <mesh
-          filename="package://roborts_gazebo/meshes/Front_Right_Wheel.STL" />
+        rpy="1.5708 0 1.5708" />
+      <geometry>
+        <mesh filename="package://roborts_gazebo/meshes/Front_Right_Wheel.STL" />
       </geometry>
     </collision>
   </link>
-  <joint
-    name="Front_Right_Wheel_Joint"
+  <joint name="base_link_to_fr_wheel_joint" type="fixed">
+    <origin
+      xyz="0.21206 0.1609 0.0022"
+      rpy="6.9321E-17 -3.6891E-17 -3.1416" />
+    <parent link="base_link" />
+    <child link="fr_wheel_Link" />
+  </joint>
+  <link name="br_wheel_Link">
+    <inertial>
+      <origin
+        xyz="-5.2323E-06 -0.014549 -9.0423E-06"
+        rpy="0 0 0" />
+      <mass value="0.86078" />
+      <inertia
+        ixx="0.0015361"
+        ixy="1.6481E-06"
+        ixz="-2.0131E-06"
+        iyy="0.002844"
+        iyz="-9.4912E-07"
+        izz="0.0015338" />
+    </inertial>
+    <visual>
+      <origin
+        xyz="0 0 0"
+        rpy="1.5708 0 1.5708"/>
+      <geometry>
+        <mesh filename="package://roborts_gazebo/meshes/Rear_Right_Wheel.STL" />
+      </geometry>
+      <material name="">
+        <color rgba="0.79216 0.81961 0.93333 1" />
+      </material>
+    </visual>
+    <collision>
+      <origin
+        xyz="0 0 0"
+        rpy="1.5708 0 1.5708"/>
+      <geometry>
+        <mesh filename="package://roborts_gazebo/meshes/Rear_Right_Wheel.STL" />
+      </geometry>
+    </collision>
+  </link>
+  <joint name="base_link_to_br_wheel_joint" type="fixed">
+    <origin
+      xyz="-0.21194 0.1603 0.0022"
+      rpy="5.7896E-17 1.5832E-16 3.1416" />
+    <parent link="base_link" />
+    <child link="br_wheel_Link" />
+  </joint>
+  <link name="bl_wheel_Link">
+    <inertial>
+      <origin
+        xyz="0.00010086 0.014592 4.8286E-05"
+        rpy="0 0 0" />
+      <mass
+        value="0.86078" />
+      <inertia
+        ixx="0.0015355"
+        ixy="5.3543E-07"
+        ixz="1.8067E-06"
+        iyy="0.002844"
+        iyz="1.1717E-07"
+        izz="0.0015337" />
+    </inertial>
+    <visual>
+      <origin
+        xyz="0 0 0"
+        rpy="1.5708 0 1.5708"/>
+      <geometry>
+        <mesh
+          filename="package://roborts_gazebo/meshes/Rear_Left_Wheel.STL" />
+      </geometry>
+      <material
+        name="">
+        <color
+          rgba="0.75294 0.75294 0.75294 1" />
+      </material>
+    </visual>
+    <collision>
+      <origin
+        xyz="0 0 0"
+        rpy="1.5708 0 1.5708"/>
+      <geometry>
+        <mesh
+          filename="package://roborts_gazebo/meshes/Rear_Left_Wheel.STL" />
+      </geometry>
+    </collision>
+  </link>
+  <joint
+    name="base_link_to_bl_wheel_joint"
     type="fixed">
     <origin
-      xyz="-0.084088 0.020672 0.74645"
-      rpy="1.5708 0 0" />
+      xyz="-0.21206 -0.1703 0.0022"
+      rpy="4.8881E-16 -3.6891E-17 -3.1416" />
     <parent
       link="base_link" />
     <child
-      link="Front_Right_Wheel" />
-    <axis
-      xyz="1 0 0" />
-    <limit
-      effort="0"
-      velocity="0" />
-  </joint>
-  <link
-    name="Front_Left_Wheel">
-    <inertial>
-      <origin
-        xyz="0.024147 -1.0711E-05 5.6176E-05"
-        rpy="0 0 0" />
-      <mass
-        value="0.21911" />
-      <inertia
-        ixx="0.00087242"
-        ixy="9.7827E-09"
-        ixz="2.3932E-07"
-        iyy="0.00045756"
-        iyz="8.8102E-08"
-        izz="0.0004578" />
-    </inertial>
-    <visual>
-      <origin
-        xyz="0 0 0"
-        rpy="0 0 0" />
-      <geometry>
-        <mesh
-          filename="package://roborts_gazebo/meshes/Front_Left_Wheel.STL" />
-      </geometry>
-      <material
-        name="">
-        <color
-          rgba="0.79216 0.81961 0.93333 1" />
-      </material>
-    </visual>
-    <collision>
-      <origin
-        xyz="0 0 0"
-        rpy="0 0 0" />
-      <geometry>
-        <mesh
-          filename="package://roborts_gazebo/meshes/Front_Left_Wheel.STL" />
-      </geometry>
-    </collision>
-  </link>
-  <joint
-    name="Front_Left_Wheel_Joint"
-    type="fixed">
-    <origin
-      xyz="0.26361 0.020672 0.74645"
-      rpy="1.5708 0 0" />
-    <parent
-      link="base_link" />
-    <child
-      link="Front_Left_Wheel" />
-    <axis
-      xyz="1 0 0" />
-    <limit
-      effort="0"
-      velocity="0" />
-  </joint>
-  <link
-    name="Rear_Right_Wheel">
-    <inertial>
-      <origin
-        xyz="-0.023927 -4.8934E-06 -4.7019E-07"
-        rpy="0 0 0" />
-      <mass
-        value="0.21911" />
-      <inertia
-        ixx="0.00087242"
-        ixy="-2.3408E-08"
-        ixz="2.3652E-07"
-        iyy="0.00045739"
-        iyz="-5.761E-08"
-        izz="0.00045797" />
-    </inertial>
-    <visual>
-      <origin
-        xyz="0 0 0"
-        rpy="0 0 0" />
-      <geometry>
-        <mesh
-          filename="package://roborts_gazebo/meshes/Rear_Right_Wheel.STL" />
-      </geometry>
-      <material
-        name="">
-        <color
-          rgba="0.79216 0.81961 0.93333 1" />
-      </material>
-    </visual>
-    <collision>
-      <origin
-        xyz="0 0 0"
-        rpy="0 0 0" />
-      <geometry>
-        <mesh
-          filename="package://roborts_gazebo/meshes/Rear_Right_Wheel.STL" />
-      </geometry>
-    </collision>
-  </link>
-  <joint
-    name="Rear_Right_Wheel_Joint"
-    type="fixed">
-    <origin
-      xyz="-0.084088 0.020672 0.33145"
-      rpy="1.5708 0 0" />
-    <parent
-      link="base_link" />
-    <child
-      link="Rear_Right_Wheel" />
-    <axis
-      xyz="1 0 0" />
-    <limit
-      effort="0"
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