Commit message: update ros old

File: Ros_old/roborts/roborts_gazebo/urdf/roborts.gazebo.xacro (robot description, xacro)
@@ -22,12 +22,24 @@
     <turnGravityOff>false</turnGravityOff>
   </gazebo>
-  <!--<gazebo reference="base_laser_link">
-    <material>Gazebo/Orange</material>
+  <gazebo reference="base_laser_link">
+    <material>Gazebo/Gray</material>
     <turnGravityOff>false</turnGravityOff>
   </gazebo>
-  <gazebo reference="led_Link">
+  <gazebo reference="front_led_Link">
     <material>Gazebo/Red</material>
     <turnGravityOff>false</turnGravityOff>
-  </gazebo>-->
+  </gazebo>
+  <gazebo reference="right_led_Link">
+    <material>Gazebo/Red</material>
+    <turnGravityOff>false</turnGravityOff>
+  </gazebo>
+  <gazebo reference="left_led_Link">
+    <material>Gazebo/Red</material>
+    <turnGravityOff>false</turnGravityOff>
+  </gazebo>
+  <gazebo reference="hp_led_Link">
+    <material>Gazebo/Red</material>
+    <turnGravityOff>false</turnGravityOff>
+  </gazebo>
   <gazebo reference="yaw_Link">
     <material>Gazebo/Red</material>
@@ -38,5 +50,5 @@
                That pixel's noise value is added to each of its color
                channels, which at that point lie in the range [0,1]. -->
-  <!--<gazebo reference="base_laser_link">
+  <gazebo reference="base_laser_link">
     <sensor type="ray" name="head_hokuyo_sensor">
       <pose>2000 2000 2000 0 0 0</pose>
@@ -69,5 +81,5 @@
     </sensor>
   </gazebo>
-  <gazebo>
+ <!-- <gazebo>
     <plugin name="realsense_plugin" filename="libRealSensePlugin.so"/>
   </gazebo>

File: Ros_old/roborts/roborts_gazebo/urdf/roborts.xacro (robot description, xacro)
@@ -425,9 +425,4 @@
           filename="package://roborts_gazebo/meshes/realsense.dae" />
       </geometry>
-      <material
-        name="">
-        <color
-          rgba="0.75294 0.75294 0.75294 1" />
-      </material>
     </visual>
     <!--<collision>
@@ -454,5 +449,4 @@
       xyz="0 0 0" />
   </joint>
-<!--
   <link
     name="base_laser_link">
@@ -477,5 +471,5 @@
       <geometry>
         <mesh
-          filename="package://roborts_gazebo/meshes/rplidar_main.STL" />
+          filename="package://roborts_gazebo/meshes/test_a2.stl" scale="0.001 0.001 0.001"/>
       </geometry>
       <material
@@ -485,13 +479,13 @@
       </material>
     </visual>
-    <collision>
-      <origin
-        xyz="0 0 0"
-        rpy="0 0 0" />
-      <geometry>
-        <mesh
-          filename="package://roborts_gazebo/meshes/rplidar_main.STL" />
-      </geometry>
-    </collision>
+    <!--<collision>
+      <origin
+        xyz="0 0 0"
+        rpy="0 0 0" />
+      <geometry>
+        <mesh
+          filename="package://roborts_gazebo/meshes/rplidar-a2m4-r1.STL" scale="0.001 0.001 0.001"/>
+      </geometry>
+    </collision>-->
   </link>
   <joint
@@ -499,6 +493,6 @@
     type="fixed">
     <origin
-      xyz="0.17456 0 0.1042"
-      rpy="4.8881E-16 -3.6891E-17 -3.1416" />
+      xyz="0.16 -0.08 0.1"
+      rpy="1.57 0 3.14" />
     <parent
       link="base_link" />
@@ -509,5 +503,5 @@
   </joint>
   <link
-    name="led_Link">
+    name="right_led_Link">
     <inertial>
       <origin
@@ -530,6 +524,59 @@
       <geometry>
         <mesh
+          filename="package://roborts_gazebo/meshes/right_led_part.STL" scale="0.001 0.001 0.001"/>
+      </geometry>
+      <material
+        name="">
+        <color
+          rgba="1 0 0 1" />
+      </material>
+    </visual>
+    <!--<collision>
+      <origin
+        xyz="0 0 0"
+        rpy="0 0 0" />
+      <geometry>
+        <mesh
           filename="package://roborts_gazebo/meshes/led_Link.STL" />
       </geometry>
+    </collision>-->
+  </link>
+  <joint
+    name="base_link_to_right_led_joint"
+    type="fixed">
+    <origin
+      xyz="-0.07 -0.205 0.08"
+      rpy="-3.14 0 1.57" />
+    <parent
+      link="base_link" />
+    <child
+      link="right_led_Link" />
+    <axis
+      xyz="0 0 0" />
+  </joint>
+  <link
+    name="left_led_Link">
+    <inertial>
+      <origin
+        xyz="-0.27282 -0.063339 0.010089"
+        rpy="0 0 0" />
+      <mass
+        value="0.028183" />
+      <inertia
+        ixx="0.00037048"
+        ixy="7.803E-06"
+        ixz="9.4378E-05"
+        iyy="0.0011379"
+        iyz="-1.4266E-06"
+        izz="0.0014674" />
+    </inertial>
+    <visual>
+      <origin
+        xyz="0 0 0"
+        rpy="0 0 0" />
+      <geometry>
+        <mesh
+          filename="package://roborts_gazebo/meshes/left_led_part.STL" scale="0.001 0.001 0.001"/>
+      </geometry>
       <material
         name="">
@@ -538,26 +585,132 @@
       </material>
     </visual>
-    <collision>
-      <origin
-        xyz="0 0 0"
-        rpy="0 0 0" />
-      <geometry>
-        <mesh
-          filename="package://roborts_gazebo/meshes/led_Link.STL" />
-      </geometry>
-    </collision>
-  </link>
-  <joint
-    name="base_link_to_led_joint"
-    type="fixed">
-    <origin
-      xyz="-0.28244 -0.063339 0.061918"
-      rpy="1.0523E-16 2.5064E-17 3.1416" />
+    <!--<collision>
+      <origin
+        xyz="0 0 0"
+        rpy="0 0 0" />
+      <geometry>
+        <mesh
+          filename="package://roborts_gazebo/meshes/left_led_Link.STL" />
+      </geometry>
+    </collision>-->
+  </link>
+  <joint
+    name="base_link_to_left_led_joint"
+    type="fixed">
+    <origin
+      xyz="-0.07 0 0.08"
+      rpy="-3.14 0 1.57" />
     <parent
       link="base_link" />
     <child
-      link="led_Link" />
+      link="left_led_Link" />
     <axis
       xyz="0 0 0" />
-  </joint>-->
+  </joint>
+  <link
+    name="hp_led_Link">
+    <inertial>
+      <origin
+        xyz="-0.27282 -0.063339 0.010089"
+        rpy="0 0 0" />
+      <mass
+        value="0.028183" />
+      <inertia
+        ixx="0.00037048"
+        ixy="7.803E-06"
+        ixz="9.4378E-05"
+        iyy="0.0011379"
+        iyz="-1.4266E-06"
+        izz="0.0014674" />
+    </inertial>
+    <visual>
+      <origin
+        xyz="0 0 0"
+        rpy="0 0 0" />
+      <geometry>
+        <mesh
+          filename="package://roborts_gazebo/meshes/hp_led_part.STL" scale="0.001 0.001 0.001"/>
+      </geometry>
+      <material
+        name="">
+        <color
+          rgba="1 0 0 1" />
+      </material>
+    </visual>
+    <!--<collision>
+      <origin
+        xyz="0 0 0"
+        rpy="0 0 0" />
+      <geometry>
+        <mesh
+          filename="package://roborts_gazebo/meshes/left_led_Link.STL" />
+      </geometry>
+    </collision>-->
+  </link>
+  <joint
+    name="base_link_to_hp_led_joint"
+    type="fixed">
+    <origin
+      xyz="-0.23 -0.14 0.18"
+      rpy="-3.14 0 1.57" />
+    <parent
+      link="base_link" />
+    <child
+      link="hp_led_Link" />
+    <axis
+      xyz="0 0 0" />
+  </joint>
+  <link
+    name="front_led_Link">
+    <inertial>
+      <origin
+        xyz="-0.27282 -0.063339 0.010089"
+        rpy="0 0 0" />
+      <mass
+        value="0.028183" />
+      <inertia
+        ixx="0.00037048"
+        ixy="7.803E-06"
+        ixz="9.4378E-05"
+        iyy="0.0011379"
+        iyz="-1.4266E-06"
+        izz="0.0014674" />
+    </inertial>
+    <visual>
+      <origin
+        xyz="0 0 0"
+        rpy="0 0 0" />
+      <geometry>
+        <mesh
+          filename="package://roborts_gazebo/meshes/front_led_part.STL" scale="0.001 0.001 0.001"/>
+      </geometry>
+      <material
+        name="">
+        <color
+          rgba="1 0 0 1" />
+      </material>
+    </visual>
+    <!--<collision>
+      <origin
+        xyz="0 0 0"
+        rpy="0 0 0" />
+      <geometry>
+        <mesh
+          filename="package://roborts_gazebo/meshes/left_led_Link.STL" />
+      </geometry>
+    </collision>-->
+  </link>
+  <joint
+    name="base_link_to_front_led_joint"
+    type="fixed">
+    <origin
+      xyz="0.175 -0.075 0.082"
+      rpy="-3.14 0 1.57" />
+    <parent
+      link="base_link" />
+    <child
+      link="front_led_Link" />
+    <axis
+      xyz="0 0 0" />
+  </joint>
 </robot>

Commit message: update ros old

File: Ros_old/roborts/roborts_gazebo/urdf/roborts.gazebo.xacro (robot description, xacro)
@@ -3,5 +3,5 @@
   <!-- materials -->
   <gazebo reference="base_link">
-    <material>Gazebo/Black</material>
+    <material>Gazebo/Grey</material>
     <turnGravityOff>false</turnGravityOff>
   </gazebo>
@@ -23,5 +23,5 @@
   </gazebo>
   <gazebo reference="base_laser_link">
-    <material>Gazebo/Gray</material>
+    <material>Gazebo/Blue</material>
     <turnGravityOff>false</turnGravityOff>
   </gazebo>
@@ -43,5 +43,9 @@
   </gazebo>
   <gazebo reference="yaw_Link">
-    <material>Gazebo/Red</material>
+    <material>Gazebo/Orange</material>
+    <turnGravityOff>false</turnGravityOff>
+  </gazebo>
+  <gazebo reference="pitch_Link">
+    <material>Gazebo/Orange</material>
     <turnGravityOff>false</turnGravityOff>
   </gazebo>
@@ -60,11 +64,11 @@
             <samples>720</samples>
             <resolution>1</resolution>
-            <min_angle>-1.570796</min_angle>
-            <max_angle>1.570796</max_angle>
+            <min_angle>-2.3</min_angle>
+            <max_angle>2.3</max_angle>
           </horizontal>
         </scan>
         <range>
           <min>0.10</min>
-          <max>30.0</max>
+          <max>10.0</max>
           <resolution>0.01</resolution>
         </range>
@@ -81,43 +85,7 @@
     </sensor>
   </gazebo>
-  <gazebo>
+  <!--<gazebo>
     <plugin name="realsense_plugin" filename="libRealSensePlugin.so"/>
-  </gazebo>
-  <!--<gazebo reference="camera_Link">
-    <sensor type="camera" name="camera1">
-      <update_rate>30.0</update_rate>
-      <camera name="head">
-        <horizontal_fov>1.3962634</horizontal_fov>
-        <image>
-          <width>800</width>
-          <height>800</height>
-          <format>R8G8B8</format>
-        </image>
-        <clip>
-          <near>0.02</near>
-          <far>300</far>
-        </clip>
-        <noise>
-          <type>gaussian</type>
-          <mean>0.0</mean>
-          <stddev>0.007</stddev>
-        </noise>
-      </camera>
-      <plugin name="camera_controller" filename="libgazebo_ros_camera.so">
-        <alwaysOn>true</alwaysOn>
-        <updateRate>0.0</updateRate>
-        <cameraName>robot/camera1</cameraName>
-        <imageTopicName>image_raw</imageTopicName>
-        <cameraInfoTopicName>camera_info</cameraInfoTopicName>
-        <frameName>camera_Link</frameName>
-        <hackBaseline>0.07</hackBaseline>
-        <distortionK1>0.0</distortionK1>
-        <distortionK2>0.0</distortionK2>
-        <distortionK3>0.0</distortionK3>
-        <distortionT1>0.0</distortionT1>
-        <distortionT2>0.0</distortionT2>
-      </plugin>
-    </sensor>
-  </gazebo>  -->
+  </gazebo>-->
   <!-- position controller plugin-->
   <gazebo>
@@ -144,5 +112,5 @@
       <reference_frame>map</reference_frame>
       <force>4000.0</force>
-      <default_freq>10</default_freq>
+      <default_freq>30</default_freq>
     </plugin>
   </gazebo>

File: Ros_old/roborts/roborts_gazebo/urdf/roborts.xacro (robot description, xacro)
@@ -72,8 +72,8 @@
     <collision>
       <origin
-        xyz="0 0 0"
-        rpy="1.5708 0 1.5708"/>
-      <geometry>
-        <mesh filename="package://roborts_gazebo/meshes/Front_Left_Wheel.STL" />
+        xyz="0 0.01 0"
+        rpy="1.5708 0 0" />
+      <geometry>
+        <cylinder radius="0.075" length="0.04"/>
       </geometry>
     </collision>
@@ -115,8 +115,8 @@
     <collision>
       <origin
-        xyz="0 0 0"
-        rpy="1.5708 0 1.5708" />
-      <geometry>
-        <mesh filename="package://roborts_gazebo/meshes/Front_Right_Wheel.STL" />
+        xyz="0 -0.01 0"
+        rpy="1.5708 0 0" />
+      <geometry>
+        <cylinder radius="0.075" length="0.04"/>
       </geometry>
     </collision>
@@ -156,8 +156,8 @@
     <collision>
       <origin
-        xyz="0 0 0"
-        rpy="1.5708 0 1.5708"/>
-      <geometry>
-        <mesh filename="package://roborts_gazebo/meshes/Rear_Right_Wheel.STL" />
+        xyz="0 -0.01 0"
+        rpy="1.5708 0 0" />
+      <geometry>
+        <cylinder radius="0.075" length="0.04"/>
       </geometry>
     </collision>
@@ -201,9 +201,8 @@
     <collision>
       <origin
-        xyz="0 0 0"
-        rpy="1.5708 0 1.5708"/>
-      <geometry>
-        <mesh
-          filename="package://roborts_gazebo/meshes/Rear_Left_Wheel.STL" />
+        xyz="0 0.01 0"
+        rpy="1.5708 0 0" />
+      <geometry>
+        <cylinder radius="0.075" length="0.04"/>
       </geometry>
     </collision>
@@ -220,5 +219,5 @@
       link="bl_wheel_Link" />
   </joint>
-    <link
+  <link
     name="Projector_Bottom">
     <inertial>
@@ -250,13 +249,4 @@
       </material>
     </visual>
-    <!--<collision>
-      <origin
-        xyz="0 0 0"
-        rpy="1.5708 0 1.5708" />
-      <geometry>
-        <mesh
-          filename="package://roborts_gazebo/meshes/Projector_Bottom.STL" />
-      </geometry>
-    </collision>-->
   </link>
   <joint
@@ -303,13 +293,4 @@
       </material>
     </visual>
-    <!--<collision>
-      <origin
-        xyz="0 0 0"
-        rpy="0 0 0" />
-      <geometry>
-        <mesh
-          filename="package://roborts_gazebo/meshes/Projector_Middle.STL" />
-      </geometry>
-    </collision>-->
   </link>
   <joint
@@ -391,5 +372,5 @@
       <inertia ixx="0.0004"  ixy="0"  ixz="0" iyy="0.0004" iyz="0" izz="0.0004" />
     </inertial>
-    <visual>
+    <!--<visual>
       <origin xyz="0 0 0" rpy="0 0 0"/>
       <geometry>
@@ -399,5 +380,5 @@
         <color rgba="1.0 1.0 1.0 1.0"/>
       </material>
-    </visual>
+    </visual>-->
   </link>
   <link
@@ -467,6 +448,6 @@
     <visual>
       <origin
-        xyz="0 0 0"
-        rpy="0 0 0" />
+      xyz="0 -0.08 -0.03"
+      rpy="1.57 0 3.14" />
       <geometry>
         <mesh
@@ -479,13 +460,4 @@
       </material>
     </visual>
-    <!--<collision>
-      <origin
-        xyz="0 0 0"
-        rpy="0 0 0" />
-      <geometry>
-        <mesh
-          filename="package://roborts_gazebo/meshes/rplidar-a2m4-r1.STL" scale="0.001 0.001 0.001"/>
-      </geometry>
-    </collision>-->
   </link>
   <joint
@@ -493,6 +465,6 @@
     type="fixed">
     <origin
-      xyz="0.16 -0.08 0.1"
-      rpy="1.57 0 3.14" />
+      xyz="0.16 0 0.12"
+      rpy="0 0 0" />
     <parent
       link="base_link" />
@@ -532,13 +504,4 @@
       </material>
     </visual>
-    <!--<collision>
-      <origin
-        xyz="0 0 0"
-        rpy="0 0 0" />
-      <geometry>
-        <mesh
-          filename="package://roborts_gazebo/meshes/led_Link.STL" />
-      </geometry>
-    </collision>-->
   </link>
   <joint
@@ -585,13 +548,4 @@
       </material>
     </visual>
-    <!--<collision>
-      <origin
-        xyz="0 0 0"
-        rpy="0 0 0" />
-      <geometry>
-        <mesh
-          filename="package://roborts_gazebo/meshes/left_led_Link.STL" />
-      </geometry>
-    </collision>-->
   </link>
   <joint
@@ -638,13 +592,4 @@
       </material>
     </visual>
-    <!--<collision>
-      <origin
-        xyz="0 0 0"
-        rpy="0 0 0" />
-      <geometry>
-        <mesh
-          filename="package://roborts_gazebo/meshes/left_led_Link.STL" />
-      </geometry>
-    </collision>-->
   </link>
   <joint
@@ -691,13 +636,4 @@
       </material>
     </visual>
-    <!--<collision>
-      <origin
-        xyz="0 0 0"
-        rpy="0 0 0" />
-      <geometry>
-        <mesh
-          filename="package://roborts_gazebo/meshes/left_led_Link.STL" />
-      </geometry>
-    </collision>-->
   </link>
   <joint
