Commit message: update roborts

File: Roborts/roborts_gazebo/urdf/roborts.base.xacro (robot description, xacro)
@@ -32,5 +32,5 @@
       </material>
     </visual>
-    <collision>
+    <!--<collision>
       <origin
         xyz="0 0 0.05"
@@ -39,5 +39,5 @@
         <box size="0.5 0.3 0.16" />
       </geometry>
-    </collision>
+    </collision>-->
   </link>
   <link name="fl_wheel_Link">
@@ -649,3 +649,47 @@
       xyz="0 0 0" />
   </joint>
+  <link
+    name="back_led_Link">
+    <inertial>
+      <origin
+        xyz="-0.27282 -0.063339 0.010089"
+        rpy="0 0 0" />
+      <mass
+        value="0.028183" />
+      <inertia
+        ixx="0.00037048"
+        ixy="7.803E-06"
+        ixz="9.4378E-05"
+        iyy="0.0011379"
+        iyz="-1.4266E-06"
+        izz="0.0014674" />
+    </inertial>
+    <visual>
+      <origin
+        xyz="0 0 0"
+        rpy="0 0 0" />
+      <geometry>
+        <mesh
+          filename="package://roborts_gazebo/meshes/back_led_part.STL" scale="0.001 0.001 0.001"/>
+      </geometry>
+      <material
+        name="">
+        <color
+          rgba="1 0 0 1" />
+      </material>
+    </visual>
+  </link>
+  <joint
+    name="base_link_to_back_led_joint"
+    type="fixed">
+    <origin
+      xyz="-0.275 -0.075 0.082"
+      rpy="-3.14 0 1.57" />
+    <parent
+      link="base_link" />
+    <child
+      link="back_led_Link" />
+    <axis
+      xyz="0 0 0" />
+  </joint>
 </robot>

File: Roborts/roborts_gazebo/urdf/roborts.gazebo.xacro (robot description, xacro)
@@ -51,5 +51,20 @@
       <turnGravityOff>false</turnGravityOff>
     </gazebo>
+    <gazebo reference="back_led_Link">
+      <material>Gazebo/${led_color}</material>
+      <turnGravityOff>false</turnGravityOff>
+    </gazebo>
   </xacro:macro>
+  <!-- position controller plugin-->
+  <gazebo>
+    <plugin name="mecanum_base_controller" filename="libgazebo_ros_planar_move.so">
+      <commandTopic>cmd_vel</commandTopic>
+      <odometryTopic>odom</odometryTopic>
+      <odometryFrame>odom</odometryFrame>
+      <odometryRate>100.0</odometryRate>
+      <robotBaseFrame>base_footprint</robotBaseFrame>
+      <broadcastTF>true</broadcastTF>
+  </plugin>
+</gazebo>
   <xacro:macro name="gazebo_plugin" params="namespace">
     <!-- hokuyo -->
@@ -91,15 +106,4 @@
       <plugin name="realsense_plugin" filename="libRealSensePlugin.so"/>
     </gazebo>-->
-    <!-- position controller plugin-->
-    <gazebo>
-      <plugin name="mecanum_base_controller" filename="libgazebo_ros_planar_move.so">
-        <commandTopic>cmd_vel</commandTopic>
-        <odometryTopic>odom</odometryTopic>
-        <odometryFrame>odom</odometryFrame>
-        <odometryRate>100.0</odometryRate>
-        <robotBaseFrame>base_footprint</robotBaseFrame>
-        <broadcastTF>true</broadcastTF>
-    </plugin>
-  </gazebo>
     <gazebo>
       <plugin name="gazebo_ros_control" filename="libgazebo_ros_control.so">
@@ -114,5 +118,5 @@
         <gimbal_link>${namespace}/pitch_Link</gimbal_link>
         <fake_link>${namespace}/fake_link</fake_link>
-        <reference_frame>${namespace}/map</reference_frame>
+        <reference_frame>map</reference_frame>
         <force>4000.0</force>
         <default_freq>30</default_freq>

Commit message: add armor contact sensor in gazebo

File: Roborts/roborts_gazebo/urdf/roborts.base.xacro (robot description, xacro)
@@ -32,12 +32,12 @@
       </material>
     </visual>
-    <!--<collision>
-      <origin
-        xyz="0 0 0.05"
-        rpy="0 0 0" />
-      <geometry>
-        <box size="0.5 0.3 0.16" />
-      </geometry>
-    </collision>-->
+    <collision name="base_link_bump_sensor_collision">
+      <origin
+        xyz="-0.1 0 0.05"
+        rpy="0 0 0" />
+      <geometry>
+        <box size="0.25 0.3 0.16" />
+      </geometry>
+    </collision>
   </link>
   <link name="fl_wheel_Link">
@@ -693,3 +693,159 @@
       xyz="0 0 0" />
   </joint>
+  <link
+    name="front_armor_link">
+    <inertial>
+      <origin
+        xyz="-0.27282 -0.063339 0.010089"
+        rpy="0 0 0" />
+      <mass
+        value="0.028183" />
+      <inertia
+        ixx="0.00037048"
+        ixy="7.803E-06"
+        ixz="9.4378E-05"
+        iyy="0.0011379"
+        iyz="-1.4266E-06"
+        izz="0.0014674" />
+    </inertial>
+    <collision name="front_armor_collision">
+      <origin
+        xyz="0 0 0"
+        rpy="0 0 0" />
+      <geometry>
+        <mesh
+          filename="package://roborts_gazebo/meshes/back_armor.STL"/>
+      </geometry>
+    </collision>
+  </link>
+  <joint
+    name="base_link_to_front_armor_joint"
+    type="fixed">
+    <origin
+      xyz="0.28 0.04 0.0"
+      rpy="0 0 1.57" />
+    <parent
+      link="base_link" />
+    <child
+      link="front_armor_link" />
+    <axis
+      xyz="0 0 0" />
+  </joint>
+  <link
+    name="left_armor_link">
+    <inertial>
+      <origin
+        xyz="-0.27282 -0.063339 0.010089"
+        rpy="0 0 0" />
+      <mass
+        value="0.028183" />
+      <inertia
+        ixx="0.00037048"
+        ixy="7.803E-06"
+        ixz="9.4378E-05"
+        iyy="0.0011379"
+        iyz="-1.4266E-06"
+        izz="0.0014674" />
+    </inertial>
+    <collision name="left_armor_collision">
+      <origin
+        xyz="0 0 0"
+        rpy="0 0 0" />
+      <geometry>
+        <mesh
+          filename="package://roborts_gazebo/meshes/left_armor.STL"/>
+      </geometry>
+    </collision>
+  </link>
+  <joint
+    name="base_link_to_left_armor_joint"
+    type="fixed">
+    <origin
+      xyz="-0.05 0.16 0.1"
+      rpy="3.14 0 1.57" />
+    <parent
+      link="base_link" />
+    <child
+      link="left_armor_link" />
+    <axis
+      xyz="0 0 0" />
+  </joint>
+  <link
+    name="right_armor_link">
+    <inertial>
+      <origin
+        xyz="-0.27282 -0.063339 0.010089"
+        rpy="0 0 0" />
+      <mass
+        value="0.028183" />
+      <inertia
+        ixx="0.00037048"
+        ixy="7.803E-06"
+        ixz="9.4378E-05"
+        iyy="0.0011379"
+        iyz="-1.4266E-06"
+        izz="0.0014674" />
+    </inertial>
+    <collision name="right_armor_collision">
+      <origin
+        xyz="0 0 0"
+        rpy="0 0 0" />
+      <geometry>
+        <mesh
+          filename="package://roborts_gazebo/meshes/right_armor.STL"/>
+      </geometry>
+    </collision>
+  </link>
+  <joint
+    name="base_link_to_right_armor_joint"
+    type="fixed">
+    <origin
+      xyz="0.045 -0.145 0.09"
+      rpy="3.14 0 1.57" />
+    <parent
+      link="base_link" />
+    <child
+      link="right_armor_link" />
+    <axis
+      xyz="0 0 0" />
+  </joint>
+  <link
+    name="back_armor_link">
+    <inertial>
+      <origin
+        xyz="-0.27282 -0.063339 0.010089"
+        rpy="0 0 0" />
+      <mass
+        value="0.028183" />
+      <inertia
+        ixx="0.00037048"
+        ixy="7.803E-06"
+        ixz="9.4378E-05"
+        iyy="0.0011379"
+        iyz="-1.4266E-06"
+        izz="0.0014674" />
+    </inertial>
+    <collision name="back_armor_collision">
+      <origin
+        xyz="0 0 0"
+        rpy="0 0 0" />
+      <geometry>
+        <mesh
+          filename="package://roborts_gazebo/meshes/back_armor.STL"/>
+      </geometry>
+    </collision>
+  </link>
+  <joint
+    name="base_link_to_back_armor_joint"
+    type="fixed">
+    <origin
+      xyz="-0.245 -0.055 -0.005"
+      rpy="0 0 1.57" />
+    <parent
+      link="base_link" />
+    <child
+      link="back_armor_link" />
+    <axis
+      xyz="0 0 0" />
+  </joint>
 </robot>

File: Roborts/roborts_gazebo/urdf/roborts.gazebo.xacro (robot description, xacro)
@@ -123,4 +123,52 @@
       </plugin>
     </gazebo>
+    <gazebo reference="front_armor_link">
+      <sensor name="front_armor_contactsensor_sensor" type="contact">
+        <always_on>true</always_on>
+        <contact>
+          <collision>base_footprint_fixed_joint_lump__front_armor_collision_collision_6</collision>
+        </contact>
+        <plugin name="front_armor_bumper" filename="libgazebo_ros_bumper.so">
+          <bumperTopicName>front_armor_contact</bumperTopicName>
+          <frameName>front_armor_link</frameName>
+        </plugin>
+      </sensor>
+    </gazebo>
+    <gazebo reference="left_armor_link">
+      <sensor name="left_armor_contactsensor_sensor" type="contact">
+        <always_on>true</always_on>
+        <contact>
+          <collision>base_footprint_fixed_joint_lump__left_armor_collision_collision_7</collision>
+        </contact>
+        <plugin name="left_armor_bumper" filename="libgazebo_ros_bumper.so">
+          <bumperTopicName>left_armor_contact</bumperTopicName>
+          <frameName>left_armor_link</frameName>
+        </plugin>
+      </sensor>
+    </gazebo>
+    <gazebo reference="right_armor_link">
+      <sensor name="right_armor_contactsensor_sensor" type="contact">
+        <always_on>true</always_on>
+        <contact>
+          <collision>base_footprint_fixed_joint_lump__right_armor_collision_collision_8</collision>
+        </contact>
+        <plugin name="right_armor_bumper" filename="libgazebo_ros_bumper.so">
+          <bumperTopicName>right_armor_contact</bumperTopicName>
+          <frameName>right_armor_link</frameName>
+        </plugin>
+      </sensor>
+    </gazebo>
+    <gazebo reference="back_armor_link">
+      <sensor name="back_armor_contactsensor_sensor" type="contact">
+        <always_on>true</always_on>
+        <contact>
+          <collision>base_footprint_fixed_joint_lump__back_armor_collision_collision_1</collision>
+        </contact>
+        <plugin name="back_armor_bumper" filename="libgazebo_ros_bumper.so">
+          <bumperTopicName>back_armor_contact</bumperTopicName>
+          <frameName>back_armor_link</frameName>
+        </plugin>
+      </sensor>
+    </gazebo>
   </xacro:macro>
 </robot>

Commit message: add contact to robot damage msg

File: Roborts/roborts_gazebo/urdf/roborts.base.xacro (robot description, xacro)
@@ -291,6 +291,7 @@
     </visual>
   </link>
-  <joint
-    name="base_link_to_yaw_joint"
+<xacro:macro name="gimbal" params="namespace" >
+  <joint
+    name="${namespace}/base_link_to_yaw_joint"
     type="revolute">
     <origin
@@ -309,5 +310,4 @@
       velocity="100" />
   </joint>
-<xacro:macro name="gimbal" params="namespace" >
   <link
     name="${namespace}/pitch_Link">
@@ -342,5 +342,5 @@
   </link>
   <joint
-    name="base_link_to_pitch_joint"
+    name="${namespace}/base_link_to_pitch_joint"
     type="revolute">
     <origin
@@ -380,4 +380,24 @@
     </visual>-->
   </link>
+  <transmission name="${namespace}/base_link_to_yaw_joint_trans">
+    <type>transmission_interface/SimpleTransmission</type>
+    <joint name="${namespace}/base_link_to_yaw_joint">
+      <hardwareInterface>hardware_interface/EffortJointInterface</hardwareInterface>
+    </joint>
+    <actuator name="${namespace}/base_link_to_yaw_joint_motor">
+      <mechanicalReduction>1</mechanicalReduction>
+      <hardwareInterface>EffortJointInterface</hardwareInterface>
+    </actuator>
+  </transmission>
+  <transmission name="${namespace}/base_link_to_pitch_joint_trans">
+    <type>transmission_interface/SimpleTransmission</type>
+    <joint name="${namespace}/base_link_to_pitch_joint">
+      <hardwareInterface>hardware_interface/EffortJointInterface</hardwareInterface>
+    </joint>
+    <actuator name="${namespace}/base_link_to_pitch_joint_motor">
+      <mechanicalReduction>1</mechanicalReduction>
+      <hardwareInterface>EffortJointInterface</hardwareInterface>
+    </actuator>
+  </transmission>
 </xacro:macro>
   <link

File: Roborts/roborts_gazebo/urdf/roborts.gazebo.xacro (robot description, xacro)
@@ -3,34 +3,30 @@
   <!-- materials -->
   <gazebo reference="base_link">
-    <material>Gazebo/Grey</material>
+    <material>Gazebo/DarkGrey</material>
     <gravity>true</gravity>
   </gazebo>
   <gazebo reference="fr_wheel_Link">
-    <material>Gazebo/Black</material>
+    <material>Gazebo/FlatBlack</material>
     <gravity>true</gravity>
   </gazebo>
   <gazebo reference="fl_wheel_Link">
-    <material>Gazebo/Black</material>
+    <material>Gazebo/FlatBlack</material>
     <gravity>true</gravity>
   </gazebo>
   <gazebo reference="br_wheel_Link">
-    <material>Gazebo/Black</material>
+    <material>Gazebo/FlatBlack</material>
     <gravity>true</gravity>
   </gazebo>
   <gazebo reference="bl_wheel_Link">
-    <material>Gazebo/Black</material>
+    <material>Gazebo/FlatBlack</material>
     <gravity>true</gravity>
   </gazebo>
   <gazebo reference="base_laser_link">
-    <material>Gazebo/Black</material>
+    <material>Gazebo/FlatBlack</material>
     <gravity>true</gravity>
   </gazebo>
   <gazebo reference="yaw_Link">
-    <material>Gazebo/Orange</material>
+    <material>Gazebo/DarkGrey</material>
     <gravity>true</gravity>
-  </gazebo>
-  <gazebo reference="pitch_Link">
-    <material>Gazebo/Orange</material>
-    <turnGravityOff>false</turnGravityOff>
   </gazebo>
   <xacro:macro name="led_color" params="led_color">
@@ -68,4 +64,8 @@
 </gazebo>
   <xacro:macro name="gazebo_plugin" params="namespace">
+    <gazebo reference="${namespace}/pitch_Link">
+      <material>Gazebo/DarkGrey</material>
+      <turnGravityOff>false</turnGravityOff>
+    </gazebo>
     <!-- hokuyo -->
     <!-- Noise is sampled independently per pixel on each frame.

File: Roborts/roborts_gazebo/urdf/roborts.original.xacro (robot description, xacro)
@@ -2,5 +2,4 @@
 <robot xmlns:xacro="http://www.ros.org/wiki/xacro" name="roborts">
   <xacro:include filename="$(find roborts_gazebo)/urdf/roborts.gazebo.xacro"/>
-  <xacro:include filename="$(find roborts_gazebo)/urdf/roborts.trans.xacro"/>
   <xacro:include filename="$(find roborts_gazebo)/urdf/roborts.base.xacro"/>
   <xacro:property name="color" value="$(arg color)" />

File: Roborts/roborts_gazebo/urdf/roborts.xacro (robot description, xacro)
@@ -2,5 +2,4 @@
 <robot xmlns:xacro="http://www.ros.org/wiki/xacro" name="roborts">
   <xacro:include filename="$(find roborts_gazebo)/urdf/roborts.gazebo.xacro"/>
-  <xacro:include filename="$(find roborts_gazebo)/urdf/roborts.trans.xacro"/>
   <xacro:include filename="$(find roborts_gazebo)/urdf/roborts.base.xacro"/>
   <xacro:property name="color" value="$(arg color)" />

Commit message: add realsense

File: Roborts/roborts_gazebo/urdf/roborts.base.xacro (robot description, xacro)
@@ -400,5 +400,4 @@
     </actuator>
   </transmission>
-</xacro:macro>
   <link
     name="camera_Link">
@@ -426,22 +425,13 @@
       </geometry>
     </visual>
-    <!--<collision>
-      <origin
-        xyz="0 0 0"
-        rpy="0 0 0" />
-      <geometry>
-        <mesh
-          filename="package://roborts_gazebo/meshes/realsense.dae" />
-      </geometry>
-    </collision>-->
-  </link>
-  <joint
-    name="yaw_link_to_camera_wheel_joint"
-    type="fixed">
-    <origin
-      xyz="0 0.02 -0.05"
-      rpy="0 0 -1.57" />
-    <parent
-      link="yaw_Link" />
+  </link>
+  <joint
+    name="pitch_link_to_camera_wheel_joint"
+    type="fixed">
+    <origin
+      xyz="0 0.1 0.03"
+      rpy="0 0 1.57" />
+    <parent
+      link="${namespace}/pitch_Link" />
     <child
       link="camera_Link" />
@@ -449,4 +439,5 @@
       xyz="0 0 0" />
   </joint>
+</xacro:macro>
   <link
     name="base_laser_link">

File: Roborts/roborts_gazebo/urdf/roborts.gazebo.xacro (robot description, xacro)
@@ -61,6 +61,57 @@
       <robotBaseFrame>base_footprint</robotBaseFrame>
       <broadcastTF>true</broadcastTF>
-  </plugin>
-</gazebo>
+    </plugin>
+  </gazebo>
+  <gazebo>
+    <plugin name="realsense_plugin" filename="libRealSensePlugin.so"/>
+  </gazebo>
+  <!-- camera -->
+  <gazebo reference="camera_Link">
+      <sensor name="color" type="camera">
+        <pose frame="">0 -0.046 0.004 0 0 0</pose>
+        <camera name="__default__">
+          <horizontal_fov>1.047</horizontal_fov>
+          <image>
+            <width>640</width>
+            <height>480</height>
+            <format>RGB_INT8</format>
+          </image>
+          <clip>
+            <near>0.1</near>
+            <far>100</far>
+          </clip>
+          <noise>
+            <type>gaussian</type>
+            <mean>0.0</mean>
+            <stddev>0.007</stddev>
+          </noise>
+        </camera>
+        <always_on>1</always_on>
+        <update_rate>60</update_rate>
+        <visualize>1</visualize>
+      </sensor>
+      <sensor name="depth" type="depth">
+        <pose frame="">0 -0.03 0.004 0 0 0</pose>
+        <camera name="__default__">
+          <horizontal_fov>1.047</horizontal_fov>
+          <image>
+            <width>640</width>
+            <height>480</height>
+          </image>
+          <clip>
+            <near>0.1</near>
+            <far>100</far>
+          </clip>
+          <noise>
+            <type>gaussian</type>
+            <mean>0.0</mean>
+            <stddev>0.007</stddev>
+          </noise>
+        </camera>
+        <always_on>1</always_on>
+        <update_rate>60</update_rate>
+        <visualize>0</visualize>
+      </sensor>
+  </gazebo>
   <xacro:macro name="gazebo_plugin" params="namespace">
     <gazebo reference="${namespace}/pitch_Link">
@@ -103,7 +154,4 @@
       </sensor>
     </gazebo>
-    <!--<gazebo>
-      <plugin name="realsense_plugin" filename="libRealSensePlugin.so"/>
-    </gazebo>-->
     <gazebo>
       <plugin name="gazebo_ros_control" filename="libgazebo_ros_control.so">
